Commit message: merged with local changed package for rotors

File: rotors_description/urdf/crazyflie2_base.xacro (robot description, xacro)
@@ -49,14 +49,43 @@
       wait_to_record_bag="$(arg wait_to_record_bag)" />
   </xacro:if>
-  <!-- Mount a VI-sensor in front of the Firefly. -->
-  <xacro:if value="$(arg enable_vi_sensor)">
-     <xacro:vi_sensor_macro_without_visual
-      namespace="${namespace}/vi_sensor"
+  <!-- Mount a ventral camera-sensor(changed to normal cam) on the Firefly. -->
+  <xacro:if value="$(arg enable_camera_sensor)">
+     <xacro:camera_macro
+      namespace="${namespace}/ventral_cam"
       parent_link="${namespace}/base_link"
-      enable_cameras="true"
-      enable_depth="true"
-      enable_ground_truth="true">
-      <origin xyz="0.0 0.0 0.0" rpy="0.0 0.0 0.0" />
-     </xacro:vi_sensor_macro_without_visual>
+      camera_suffix="nadir"
+      frame_rate="20.0"
+      horizontal_fov="2"
+      image_width="752"
+      image_height="480"
+      image_format="R8G8B8"
+      min_distance="0.02"
+      max_distance="50"
+      noise_mean="0.0"
+      noise_stddev="0.007"
+      enable_visual="true">
+      <box size="0.005 0.005 0.002" />
+      <origin xyz="0 0 ${-arm_length/4}" rpy="0 ${pi/2} 0" />
+     </xacro:camera_macro>
+  </xacro:if>
+  <!-- Mount a frontal camera-sensor(changed to normal cam) on the Firefly. -->
+  <xacro:if value="$(arg enable_camera_sensor)">
+     <xacro:camera_macro
+      namespace="${namespace}/frontal_cam"
+      parent_link="${namespace}/base_link"
+      camera_suffix="nadir"
+      frame_rate="20.0"
+      horizontal_fov="2"
+      image_width="752"
+      image_height="480"
+      image_format="R8G8B8"
+      min_distance="0.02"
+      max_distance="50"
+      noise_mean="0.0"
+      noise_stddev="0.007"
+      enable_visual="true">
+      <box size="0.005 0.005 0.002" />
+      <origin xyz="${7*(arm_length/10)} 0 0" rpy="0 0 0" />
+     </xacro:camera_macro>
   </xacro:if>
 </robot>

File: rotors_description/urdf/firefly_base.xacro (robot description, xacro)
@@ -41,3 +41,43 @@
       wait_to_record_bag="$(arg wait_to_record_bag)" />
   </xacro:if>
+  <!-- Mount a ventral camera-sensor(changed to normal cam) on the Firefly. -->
+  <xacro:if value="$(arg enable_camera_sensor)">
+     <xacro:camera_macro
+      namespace="${namespace}/ventral_cam"
+      parent_link="${namespace}/base_link"
+      camera_suffix="nadir"
+      frame_rate="20.0"
+      horizontal_fov="2"
+      image_width="752"
+      image_height="480"
+      image_format="R8G8B8"
+      min_distance="0.02"
+      max_distance="50"
+      noise_mean="0.0"
+      noise_stddev="0.007"
+      enable_visual="true">
+      <box size="0.005 0.005 0.002" />
+      <origin xyz="0 0 ${-arm_length/4}" rpy="0 ${pi/2} 0" />
+     </xacro:camera_macro>
+  </xacro:if>
+  <!-- Mount a frontal camera-sensor(changed to normal cam) on the Firefly. -->
+  <xacro:if value="$(arg enable_camera_sensor)">
+     <xacro:camera_macro
+      namespace="${namespace}/frontal_cam"
+      parent_link="${namespace}/base_link"
+      camera_suffix="nadir"
+      frame_rate="20.0"
+      horizontal_fov="2"
+      image_width="752"
+      image_height="480"
+      image_format="R8G8B8"
+      min_distance="0.02"
+      max_distance="50"
+      noise_mean="0.0"
+      noise_stddev="0.007"
+      enable_visual="true">
+      <box size="0.005 0.005 0.002" />
+      <origin xyz="${7*(arm_length/10)} 0 0" rpy="0 0 0" />
+     </xacro:camera_macro>
+  </xacro:if>
 </robot>
