Commit message: add cam to iris model

File: rotors_description/urdf/iris_base.xacro (robot description, xacro)
@@ -23,3 +23,43 @@
       wait_to_record_bag="$(arg wait_to_record_bag)" />
   </xacro:if>
+  <!-- Mount a ventral camera-sensor(changed to normal cam) on the iris. -->
+  <xacro:if value="$(arg enable_camera_sensor)">
+     <xacro:camera_macro
+      namespace="${namespace}/ventral_cam"
+      parent_link="${namespace}/base_link"
+      camera_suffix="nadir"
+      frame_rate="20.0"
+      horizontal_fov="2"
+      image_width="752"
+      image_height="480"
+      image_format="R8G8B8"
+      min_distance="0.02"
+      max_distance="50"
+      noise_mean="0.0"
+      noise_stddev="0.007"
+      enable_visual="true">
+      <box size="0.005 0.005 0.002" />
+      <origin xyz="0 0 ${-arm_length/4}" rpy="0 ${pi/2} 0" />
+     </xacro:camera_macro>
+  </xacro:if>
+  <!-- Mount a frontal camera-sensor(changed to normal cam) on the iris. -->
+  <xacro:if value="$(arg enable_camera_sensor)">
+     <xacro:camera_macro
+      namespace="${namespace}/frontal_cam"
+      parent_link="${namespace}/base_link"
+      camera_suffix="nadir"
+      frame_rate="20.0"
+      horizontal_fov="2"
+      image_width="752"
+      image_height="480"
+      image_format="R8G8B8"
+      min_distance="0.02"
+      max_distance="50"
+      noise_mean="0.0"
+      noise_stddev="0.007"
+      enable_visual="true">
+      <box size="0.005 0.005 0.002" />
+      <origin xyz="${7*(arm_length/10)} 0 0" rpy="0 0 0" />
+     </xacro:camera_macro>
+  </xacro:if>
 </robot>

Commit message: bug fix for cam on iris

File: rotors_description/urdf/iris_base.xacro (robot description, xacro)
@@ -40,5 +40,5 @@
       enable_visual="true">
       <box size="0.005 0.005 0.002" />
-      <origin xyz="0 0 ${-arm_length/4}" rpy="0 ${pi/2} 0" />
+      <origin xyz="0 0 ${-arm_length_front_y/5}" rpy="0 ${pi/2} 0" />
      </xacro:camera_macro>
   </xacro:if>
@@ -60,5 +60,5 @@
       enable_visual="true">
       <box size="0.005 0.005 0.002" />
-      <origin xyz="${7*(arm_length/10)} 0 0" rpy="0 0 0" />
+      <origin xyz="${7*(arm_length_front_y/10)} 0 0" rpy="0 0 0" />
      </xacro:camera_macro>
   </xacro:if>

Commit message: bugfix depth sensor

File: rotors_description/urdf/iris_base.xacro (robot description, xacro)
@@ -71,5 +71,5 @@
       enable_depth="true"
       enable_ground_truth="true">
-      <origin xyz="${7*(arm_length/25)} 0 ${-arm_length/4}" rpy="0 ${pi/2} 0" />
+      <origin xyz="${7*(arm_length_front_y/25)} 0 ${-arm_length_front_y/4}" rpy="0 ${pi/2} 0" />
      </xacro:vi_sensor_macro_without_visual>
   </xacro:if>
@@ -82,5 +82,5 @@
       enable_depth="true"
       enable_ground_truth="true">
-      <origin xyz="${7*(arm_length/10)} 0 ${-arm_length/9}" rpy="0 0 0" />
+      <origin xyz="${7*(arm_length_front_y/10)} 0 ${-arm_length_front_y/9}" rpy="0 0 0" />
      </xacro:vi_sensor_macro_without_visual>
   </xacro:if>
