Commit message: add depth sensor to iris and firefly for frontend

File: rotors_description/urdf/firefly_base.xacro (robot description, xacro)
@@ -81,3 +81,25 @@
      </xacro:camera_macro>
   </xacro:if>
+  <!-- Mount a ventral VI-sensor on the Firefly. -->
+  <xacro:if value="$(arg enable_vi_sensor)">
+     <xacro:vi_sensor_macro_without_visual
+      namespace="${namespace}/vi_sensor_ventral"
+      parent_link="${namespace}/base_link"
+      enable_cameras="false"
+      enable_depth="true"
+      enable_ground_truth="true">
+      <origin xyz="${7*(arm_length/25)} 0 ${-arm_length/4}" rpy="0 ${pi/2} 0" />
+     </xacro:vi_sensor_macro_without_visual>
+  </xacro:if>
+  <!-- Mount a frontal VI-sensor on the Firefly. -->
+  <xacro:if value="$(arg enable_vi_sensor)">
+     <xacro:vi_sensor_macro_without_visual
+      namespace="${namespace}/vi_sensor_frontal"
+      parent_link="${namespace}/base_link"
+      enable_cameras="false"
+      enable_depth="true"
+      enable_ground_truth="true">
+      <origin xyz="${7*(arm_length/10)} 0 ${-arm_length/9}" rpy="0 0 0" />
+     </xacro:vi_sensor_macro_without_visual>
+  </xacro:if>
 </robot>

File: rotors_description/urdf/iris_base.xacro (robot description, xacro)
@@ -63,3 +63,25 @@
      </xacro:camera_macro>
   </xacro:if>
+  <!-- Mount a ventral VI-sensor on the Iris. -->
+  <xacro:if value="$(arg enable_vi_sensor)">
+     <xacro:vi_sensor_macro_without_visual
+      namespace="${namespace}/vi_sensor_ventral"
+      parent_link="${namespace}/base_link"
+      enable_cameras="false"
+      enable_depth="true"
+      enable_ground_truth="true">
+      <origin xyz="${7*(arm_length/25)} 0 ${-arm_length/4}" rpy="0 ${pi/2} 0" />
+     </xacro:vi_sensor_macro_without_visual>
+  </xacro:if>
+  <!-- Mount a frontal VI-sensor on the Iris. -->
+  <xacro:if value="$(arg enable_vi_sensor)">
+     <xacro:vi_sensor_macro_without_visual
+      namespace="${namespace}/vi_sensor_frontal"
+      parent_link="${namespace}/base_link"
+      enable_cameras="false"
+      enable_depth="true"
+      enable_ground_truth="true">
+      <origin xyz="${7*(arm_length/10)} 0 ${-arm_length/9}" rpy="0 0 0" />
+     </xacro:vi_sensor_macro_without_visual>
+  </xacro:if>
 </robot>

Commit message: add flashlight to iris and firefly

File: rotors_description/urdf/firefly_base.xacro (robot description, xacro)
@@ -103,3 +103,62 @@
      </xacro:vi_sensor_macro_without_visual>
   </xacro:if>
+  <xacro:if value="$(arg enable_flashlight)">
+    <gazebo>
+      <model name='flashlight'>
+        <pose>0 0 0 0 0 0</pose>
+        <link name='light_source'>
+          <pose>0 0 0.0 0.01 0 0</pose>
+          <inertial>
+            <mass>0.00000000025</mass>
+            <inertia>
+              <ixx>1.0e-012</ixx>
+              <ixy>0</ixy>
+              <ixz>0</ixz>
+              <iyy>1.0e-012</iyy>
+              <iyz>0</iyz>
+              <izz>1.0e-012</izz>
+            </inertia>
+          </inertial>
+          <light name='lamp' type='spot'>
+            <pose>0 0 0.0 0 0 0</pose>
+            <attenuation>
+              <range>0</range>
+              <linear>0</linear>
+              <constant>0.1</constant>
+              <quadratic>0.01</quadratic>
+            </attenuation>
+            <diffuse>0.8 0.8 0.5 1</diffuse>
+            <specular>0.8 0.8 0.5 1</specular>
+            <spot>
+              <inner_angle>1</inner_angle>
+              <outer_angle>1.1</outer_angle>
+              <falloff>1</falloff>
+            </spot>
+            <direction>0 0 -1</direction>
+          </light>
+          <visual name='lamp'>
+            <geometry>
+              <cylinder>
+                <radius>0.00019</radius>
+                <length>0.00005</length>
+              </cylinder>
+            </geometry>
+            <transparency>0.0</transparency>
+            <material>
+              <ambient>1 1 1 1</ambient>
+              <diffuse>1 1 1 1</diffuse>
+              <specular>1 1 1 1</specular>
+              <emissive>0.8 0.8 0.5 1</emissive>
+            </material>
+          </visual>
+        </link>
+      </model>
+    </gazebo>
+    <gazebo>
+      <joint name='flashlight_joint' type='fixed'>
+        <parent>${namespace}/base_link</parent>
+        <child>flashlight::light_source</child>
+      </joint>
+    </gazebo>
+  </xacro:if>
 </robot>

File: rotors_description/urdf/iris_base.xacro (robot description, xacro)
@@ -85,3 +85,62 @@
      </xacro:vi_sensor_macro_without_visual>
   </xacro:if>
+  <xacro:if value="$(arg enable_flashlight)">
+    <gazebo>
+      <model name='flashlight'>
+        <pose>0 0 0 0 0 0</pose>
+        <link name='light_source'>
+          <pose>0 0 0.0 0.01 0 0</pose>
+          <inertial>
+            <mass>0.00000000025</mass>
+            <inertia>
+              <ixx>1.0e-012</ixx>
+              <ixy>0</ixy>
+              <ixz>0</ixz>
+              <iyy>1.0e-012</iyy>
+              <iyz>0</iyz>
+              <izz>1.0e-012</izz>
+            </inertia>
+          </inertial>
+          <light name='lamp' type='spot'>
+            <pose>0 0 0.0 0 0 0</pose>
+            <attenuation>
+              <range>0</range>
+              <linear>0</linear>
+              <constant>0.1</constant>
+              <quadratic>0.01</quadratic>
+            </attenuation>
+            <diffuse>0.8 0.8 0.5 1</diffuse>
+            <specular>0.8 0.8 0.5 1</specular>
+            <spot>
+              <inner_angle>1</inner_angle>
+              <outer_angle>1.1</outer_angle>
+              <falloff>1</falloff>
+            </spot>
+            <direction>0 0 -1</direction>
+          </light>
+          <visual name='lamp'>
+            <geometry>
+              <cylinder>
+                <radius>0.00019</radius>
+                <length>0.00005</length>
+              </cylinder>
+            </geometry>
+            <transparency>0.0</transparency>
+            <material>
+              <ambient>1 1 1 1</ambient>
+              <diffuse>1 1 1 1</diffuse>
+              <specular>1 1 1 1</specular>
+              <emissive>0.8 0.8 0.5 1</emissive>
+            </material>
+          </visual>
+        </link>
+      </model>
+    </gazebo>
+    <gazebo>
+      <joint name='flashlight_joint' type='fixed'>
+        <parent>${namespace}/base_link</parent>
+        <child>flashlight::light_source</child>
+      </joint>
+    </gazebo>
+  </xacro:if>
 </robot>
